File: strobeGlassesMK1/_autosave-strobeGlassesMK1.kicad_sch (KiCad schematic)
At the start: 19 parts, among them J1 USB_C_Receptacle_USB2.0_14P, U1 ICM7555xB, U2 DRV8833PW, U3 MCP73871

Commit message: small updates
Parts:
- removed R1, R2: 5.1K, symbol Device:R_US
- added R10, R2, R7, R8, R9: 5.1K, symbol Device:R_Small_US
Connections:
- net GND: now also R2.2, R7.2, R8.2, R9.1
- net at J1.B5 (CC2): now also R7.1
- net at J1.A5 (CC1): now also R2.1
- net at U3.3 (SEL): now also R8.1
- net at U3.4 (PROG2): now also R9.2
- net at U3.9 (~{TE}): now also R10.1
- no-connect marks 4 -> 7
Other:
- moved on the sheet: BT1, C3, C4, D1, D2, D3, R3, R4, R5, R6, U3
